File: PCB-Kicad/Modul_Main_Board/Modul_Main_Board.kicad_pcb (KiCad board)
At the start: 2 copper layers, 80 x 100 mm, 34 parts, among them IC1 TEENSY_4.0, J1 Pixy Cam1, J10 LcdModule, J12 Screw Conn1, J13 On/Off Switch, J14 XT60-M, J15 Exposed Pins, J16 Exposed Pins, J2 Pixy Cam2, J4 HC-SR04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

Commit message: remote and pcb update
Parts:
- R1, R2, R3, R4, R5, R7, R8, R9: value 1k -> 2k
- R10: value 100 -> 220
- R6: value 1K -> 2K
Changed lines of the file:
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@@
 		(property ki_fp_filters "Connector*:*_2x??_*")
 		(sheetname "Root")
-		(sheetfile "Modul_LCD.kicad_sch")
+		(sheetfile "Modul_Main_Board.kicad_sch")
 		(attr through_hole)
 		(fp_line
@@
 			)
 		)
-		(property "Value" "1K"
+		(property "Value" "2K"
 			(at 6.35 2.92 180)
 			(layer "F.Fab")
@@
 		(property ki_fp_filters "R_*")
 		(sheetname "Root")
-		(sheetfile "Modul_LCD.kicad_sch")
+		(sheetfile "Modul_Main_Board.kicad_sch")
 		(attr through_hole)
 		(fp_line
@@
 		(property ki_fp_filters "Connector*:*_1x??_*")
 		(sheetname "Root")
-		(sheetfile "Modul_LCD.kicad_sch")
+		(sheetfile "Modul_Main_Board.kicad_sch")
 		(attr through_hole)
 		(fp_line
@@
 		(property ki_fp_filters "Connector*:*_1x??_*")
 		(sheetname "Root")
-		(sheetfile "Modul_LCD.kicad_sch")
+		(sheetfile "Modul_Main_Board.kicad_sch")
 		(attr through_hole)
 		(fp_line
@@
 			)
 		)
-		(property "Value" "1k"
+		(property "Value" "2k"
 			(at 6.35 2.92 0)
 			(layer "F.Fab")
@@
 		(property ki_fp_filters "R_*")
 		(sheetname "Root")
-		(sheetfile "Modul_LCD.kicad_sch")
+		(sheetfile "Modul_Main_Board.kicad_sch")
 		(attr through_hole)
 		(fp_line
@@
 		)
 		(sheetname "Root")
-		(sheetfile "Modul_LCD.kicad_sch")
+		(sheetfile "Modul_Main_Board.kicad_sch")
 		(attr through_hole)
 		(fp_line
@@
 		(property ki_fp_filters "MountingHole*")
 		(sheetname "Root")
-		(sheetfile "Modul_LCD.kicad_sch")
+		(sheetfile "Modul_Main_Board.kicad_sch")
 		(attr exclude_from_pos_files exclude_from_bom)
 		(fp_circle
@@
 		(property ki_fp_filters "Connector*:*_2x??_*")
 		(sheetname "Root")
-		(sheetfile "Modul_LCD.kicad_sch")
+		(sheetfile "Modul_Main_Board.kicad_sch")
 		(attr through_hole)
 		(fp_line
@@
 		)
 		(sheetname "Root")
-		(sheetfile "Modul_LCD.kicad_sch")
+		(sheetfile "Modul_Main_Board.kicad_sch")
 		(attr through_hole)
 		(fp_line
@@
 		(property ki_fp_filters "Connector*:*_1x??_*")
 		(sheetname "Root")
-		(sheetfile "Modul_LCD.kicad_sch")
+		(sheetfile "Modul_Main_Board.kicad_sch")
 		(attr through_hole)
 		(fp_line
@@
 		(property ki_fp_filters "CP_*")
 		(sheetname "Root")
-		(sheetfile "Modul_LCD.kicad_sch")
+		(sheetfile "Modul_Main_Board.kicad_sch")
 		(attr through_hole)
 		(fp_line
@@
 		)
 		(sheetname "Root")
-		(sheetfile "Modul_LCD.kicad_sch")
+		(sheetfile "Modul_Main_Board.kicad_sch")
 		(attr through_hole)
 		(fp_line
@@
 		(property ki_fp_filters "MountingHole*")
 		(sheetname "Root")
-		(sheetfile "Modul_LCD.kicad_sch")
+		(sheetfile "Modul_Main_Board.kicad_sch")
 		(attr exclude_from_pos_files exclude_from_bom)
 		(fp_circle
@@
 		(property ki_fp_filters "MountingHole*")
 		(sheetname "Root")
-		(sheetfile "Modul_LCD.kicad_sch")
+		(sheetfile "Modul_Main_Board.kicad_sch")
 		(attr exclude_from_pos_files exclude_from_bom)
 		(fp_circle
@@
 		(property ki_fp_filters "Connector*:*_1x??_*")
 		(sheetname "Root")
-		(sheetfile "Modul_LCD.kicad_sch")
+		(sheetfile "Modul_Main_Board.kicad_sch")
 		(attr through_hole)
 		(fp_line
@@
 			)
 		)
-		(property "Value" "1k"
+		(property "Value" "2k"
 			(at 6.35 2.92 180)
 			(layer "F.Fab")
@@
 		(property ki_fp_filters "R_*")
 		(sheetname "Root")
-		(sheetfile "Modul_LCD.kicad_sch")
+		(sheetfile "Modul_Main_Board.kicad_sch")
 		(attr through_hole)
 		(fp_line
@@
 			)
 		)
-		(property "Value" "1k"
+		(property "Value" "2k"
 			(at 6.35 2.92 180)
 			(layer "F.Fab")
@@
 		(property ki_fp_filters "R_*")
 		(sheetname "Root")
-		(sheetfile "Modul_LCD.kicad_sch")
+		(sheetfile "Modul_Main_Board.kicad_sch")
 		(attr through_hole)
 		(fp_line
@@
 		(property ki_fp_filters "LED* LED_SMD:* LED_THT:*")
 		(sheetname "Root")
-		(sheetfile "Modul_LCD.kicad_sch")
+		(sheetfile "Modul_Main_Board.kicad_sch")
 		(attr through_hole)
 		(fp_line
@@
 		(property ki_fp_filters "Connector*:*_1x??_*")
 		(sheetname "Root")
-		(sheetfile "Modul_LCD.kicad_sch")
+		(sheetfile "Modul_Main_Board.kicad_sch")
 		(attr through_hole)
 		(fp_line
@@
 			)
 		)
-		(property "Value" "1k"
+		(property "Value" "2k"
 			(at 6.35 2.92 0)
 			(layer "F.Fab")
@@
 		(property ki_fp_filters "R_*")
 		(sheetname "Root")
-		(sheetfile "Modul_LCD.kicad_sch")
+		(sheetfile "Modul_Main_Board.kicad_sch")
 		(attr through_hole)
 		(fp_line
@@
 		(property ki_fp_filters "MountingHole*")
 		(sheetname "Root")
-		(sheetfile "Modul_LCD.kicad_sch")
+		(sheetfile "Modul_Main_Board.kicad_sch")
 		(attr exclude_from_pos_files exclude_from_bom)
 		(fp_circle
@@
 		)
 		(sheetname "Root")
-		(sheetfile "Modul_LCD.kicad_sch")
+		(sheetfile "Modul_Main_Board.kicad_sch")
 		(attr through_hole)
 		(fp_rect
@@
 			)
 		)
-		(property "Value" "1k"
+		(property "Value" "2k"
 			(at 6.35 2.92 180)
 			(layer "F.Fab")
@@
 		(property ki_fp_filters "R_*")
 		(sheetname "Root")
-		(sheetfile "Modul_LCD.kicad_sch")
+		(sheetfile "Modul_Main_Board.kicad_sch")
 		(attr through_hole)
 		(fp_line
@@
 			)
 		)
-		(property "Value" "1k"
+		(property "Value" "2k"
 			(at 6.35 2.92 -90)
 			(layer "F.Fab")
@@
 		(property ki_fp_filters "R_*")
 		(sheetname "Root")
-		(sheetfile "Modul_LCD.kicad_sch")
+		(sheetfile "Modul_Main_Board.kicad_sch")
 		(attr through_hole)
 		(fp_line
@@
 		(property ki_fp_filters "Connector*:*_1x??_*")
 		(sheetname "Root")
-		(sheetfile "Modul_LCD.kicad_sch")
+		(sheetfile "Modul_Main_Board.kicad_sch")
 		(attr through_hole)
 		(fp_line
@@
 		(tags "Resistor Axial_DIN0411 series Axial Horizontal pin pitch 12.7mm 1W length 9.9mm diameter 3.6mm")
 		(property "Reference" "R3"
-			(at 3.85 0 360)
+			(at 3.85 0 0)
 			(layer "F.SilkS")
 			(effects
@@
 			)
 		)
-		(property "Value" "1k"
-			(at 6.35 2.92 360)
+		(property "Value" "2k"
+			(at 6.35 2.92 0)
 			(layer "F.Fab")
 			(effects
@@
 		(property ki_fp_filters "R_*")
 		(sheetname "Root")
-		(sheetfile "Modul_LCD.kicad_sch")
+		(sheetfile "Modul_Main_Board.kicad_sch")
 		(attr through_hole)
 		(fp_line
@@
 		)
 		(fp_text user "${REFERENCE}"
-			(at 6.35 0 360)
+			(at 6.35 0 0)
 			(layer "F.Fab")
 			(effects
@@
 		(property ki_fp_filters "Connector*:*_1x??_*")
 		(sheetname "Root")
-		(sheetfile "Modul_LCD.kicad_sch")
+		(sheetfile "Modul_Main_Board.kicad_sch")
 		(attr through_hole)
 		(fp_line
@@
 		(property ki_fp_filters "CP_*")
 		(sheetname "Root")
-		(sheetfile "Modul_LCD.kicad_sch")
+		(sheetfile "Modul_Main_Board.kicad_sch")
 		(attr through_hole)
 		(fp_line
@@
 		(property ki_fp_filters "Connector*:*_1x??_*")
 		(sheetname "Root")
-		(sheetfile "Modul_LCD.kicad_sch")
+		(sheetfile "Modul_Main_Board.kicad_sch")
 		(attr through_hole)
 		(fp_line
@@
 		(property ki_fp_filters "Connector*:*_1x??_*")
 		(sheetname "Root")
-		(sheetfile "Modul_LCD.kicad_sch")
+		(sheetfile "Modul_Main_Board.kicad_sch")
 		(attr through_hole)
 		(fp_line
@@
 		(property ki_fp_filters "Connector*:*_2x??_*")
 		(sheetname "Root")
-		(sheetfile "Modul_LCD.kicad_sch")
+		(sheetfile "Modul_Main_Board.kicad_sch")
 		(attr through_hole)
 		(fp_line
@@
 			)
 		)
-		(property "Value" "100"
+		(property "Value" "220"
 			(at 6.35 2.92 -90)
 			(layer "F.Fab")
@@
 		(property ki_fp_filters "R_*")
 		(sheetname "Root")
-		(sheetfile "Modul_LCD.kicad_sch")
+		(sheetfile "Modul_Main_Board.kicad_sch")
 		(attr through_hole)
 		(fp_line
@@
 			)
 		)
-		(property "Value" "1k"
+		(property "Value" "2k"
 			(at 6.35 2.92 0)
 			(layer "F.Fab")
@@
 		(property ki_fp_filters "R_*")
 		(sheetname "Root")
-		(sheetfile "Modul_LCD.kicad_sch")
+		(sheetfile "Modul_Main_Board.kicad_sch")
 		(attr through_hole)
 		(fp_line
