File: PCB-Kicad/Modul_Main_Board/Modul_Main_Board.kicad_sch (KiCad schematic)
At the start: 33 parts, among them IC1 TEENSY_4.0, J1 Pixy Cam1, J10 LcdModule, J12 Screw Conn1, J13 On/Off Switch, J14 XT60-M, J15 Exposed Pins, J16 Exposed Pins, J2 Pixy Cam2, J4 HC-SR04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

Commit message: remote and pcb update
Parts:
- R1, R2, R3, R4, R5, R7, R8, R9: value 1k -> 2k
- R10: value 100 -> 220
- R6: value 1K -> 2K
Changed lines of the file:
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@@
 		)
 		(instances
-			(project "Modul_LCD"
+			(project "Modul_Main_Board"
 				(path "/e383a7f7-29ae-4aa9-abeb-7f7854670ab9"
 					(reference "J9")
@@
 		)
 		(instances
-			(project "Modul_LCD"
+			(project "Modul_Main_Board"
 				(path "/e383a7f7-29ae-4aa9-abeb-7f7854670ab9"
 					(reference "D1")
@@
 			)
 		)
-		(property "Value" "1k"
+		(property "Value" "2k"
 			(at 34.29 44.45 90)
 			(effects
@@
 		)
 		(instances
-			(project "Modul_LCD"
+			(project "Modul_Main_Board"
 				(path "/e383a7f7-29ae-4aa9-abeb-7f7854670ab9"
 					(reference "R5")
@@
 			)
 		)
-		(property "Value" "100"
+		(property "Value" "220"
 			(at 190.5 31.75 90)
 			(effects
@@
 		)
 		(instances
-			(project "Modul_LCD"
+			(project "Modul_Main_Board"
 				(path "/e383a7f7-29ae-4aa9-abeb-7f7854670ab9"
 					(reference "R10")
@@
 		)
 		(instances
-			(project "Modul_LCD"
+			(project "Modul_Main_Board"
 				(path "/e383a7f7-29ae-4aa9-abeb-7f7854670ab9"
 					(reference "J14")
@@
 		)
 		(instances
-			(project "Modul_LCD"
+			(project "Modul_Main_Board"
 				(path "/e383a7f7-29ae-4aa9-abeb-7f7854670ab9"
 					(reference "C2")
@@
 		)
 		(instances
-			(project "Modul_LCD"
+			(project "Modul_Main_Board"
 				(path "/e383a7f7-29ae-4aa9-abeb-7f7854670ab9"
 					(reference "H3")
@@
 		)
 		(instances
-			(project "Modul_LCD"
+			(project "Modul_Main_Board"
 				(path "/e383a7f7-29ae-4aa9-abeb-7f7854670ab9"
 					(reference "J15")
@@
 		)
 		(instances
-			(project "Modul_LCD"
+			(project "Modul_Main_Board"
 				(path "/e383a7f7-29ae-4aa9-abeb-7f7854670ab9"
 					(reference "J10")
@@
 		)
 		(instances
-			(project "Modul_LCD"
+			(project "Modul_Main_Board"
 				(path "/e383a7f7-29ae-4aa9-abeb-7f7854670ab9"
 					(reference "J2")
@@
 			)
 		)
-		(property "Value" "1k"
+		(property "Value" "2k"
 			(at 26.67 44.45 90)
 			(effects
@@
 		)
 		(instances
-			(project "Modul_LCD"
+			(project "Modul_Main_Board"
 				(path "/e383a7f7-29ae-4aa9-abeb-7f7854670ab9"
 					(reference "R4")
@@
 		)
 		(instances
-			(project "Modul_LCD"
+			(project "Modul_Main_Board"
 				(path "/e383a7f7-29ae-4aa9-abeb-7f7854670ab9"
 					(reference "#G1")
@@
 			)
 		)
-		(property "Value" "1k"
+		(property "Value" "2k"
 			(at 44.45 31.75 90)
 			(effects
@@
 		)
 		(instances
-			(project "Modul_LCD"
+			(project "Modul_Main_Board"
 				(path "/e383a7f7-29ae-4aa9-abeb-7f7854670ab9"
 					(reference "R3")
@@
 			)
 		)
-		(property "Value" "1k"
+		(property "Value" "2k"
 			(at 34.29 31.75 90)
 			(effects
@@
 		)
 		(instances
-			(project "Modul_LCD"
+			(project "Modul_Main_Board"
 				(path "/e383a7f7-29ae-4aa9-abeb-7f7854670ab9"
 					(reference "R2")
@@
 		)
 		(instances
-			(project "Modul_LCD"
+			(project "Modul_Main_Board"
 				(path "/e383a7f7-29ae-4aa9-abeb-7f7854670ab9"
 					(reference "H2")
@@
 		)
 		(instances
-			(project "Modul_LCD"
+			(project "Modul_Main_Board"
 				(path "/e383a7f7-29ae-4aa9-abeb-7f7854670ab9"
 					(reference "J1")
@@
 			)
 		)
-		(property "Value" "1k"
+		(property "Value" "2k"
 			(at 26.67 57.15 90)
 			(effects
@@
 		)
 		(instances
-			(project "Modul_LCD"
+			(project "Modul_Main_Board"
 				(path "/e383a7f7-29ae-4aa9-abeb-7f7854670ab9"
 					(reference "R7")
@@
 		)
 		(instances
-			(project "Modul_LCD"
+			(project "Modul_Main_Board"
 				(path "/e383a7f7-29ae-4aa9-abeb-7f7854670ab9"
 					(reference "J13")
@@
 		)
 		(instances
-			(project "Modul_LCD"
+			(project "Modul_Main_Board"
 				(path "/e383a7f7-29ae-4aa9-abeb-7f7854670ab9"
 					(reference "IC1")
@@
 		)
 		(instances
-			(project "Modul_LCD"
+			(project "Modul_Main_Board"
 				(path "/e383a7f7-29ae-4aa9-abeb-7f7854670ab9"
 					(reference "J6")
@@
 			)
 		)
-		(property "Value" "1k"
+		(property "Value" "2k"
 			(at 44.45 57.15 90)
 			(effects
@@
 		)
 		(instances
-			(project "Modul_LCD"
+			(project "Modul_Main_Board"
 				(path "/e383a7f7-29ae-4aa9-abeb-7f7854670ab9"
 					(reference "R9")
@@
 			)
 		)
-		(property "Value" "1K"
+		(property "Value" "2K"
 			(at 44.45 44.45 90)
 			(effects
@@
 		)
 		(instances
-			(project "Modul_LCD"
+			(project "Modul_Main_Board"
 				(path "/e383a7f7-29ae-4aa9-abeb-7f7854670ab9"
 					(reference "R6")
@@
 		)
 		(instances
-			(project "Modul_LCD"
+			(project "Modul_Main_Board"
 				(path "/e383a7f7-29ae-4aa9-abeb-7f7854670ab9"
 					(reference "U1")
@@
 		)
 		(instances
-			(project "Modul_LCD"
+			(project "Modul_Main_Board"
 				(path "/e383a7f7-29ae-4aa9-abeb-7f7854670ab9"
 					(reference "H1")
@@
 		)
 		(instances
-			(project "Modul_LCD"
+			(project "Modul_Main_Board"
 				(path "/e383a7f7-29ae-4aa9-abeb-7f7854670ab9"
 					(reference "J16")
@@
 			)
 		)
-		(property "Value" "1k"
+		(property "Value" "2k"
 			(at 34.29 57.15 90)
 			(effects
@@
 		)
 		(instances
-			(project "Modul_LCD"
+			(project "Modul_Main_Board"
 				(path "/e383a7f7-29ae-4aa9-abeb-7f7854670ab9"
 					(reference "R8")
@@
 		)
 		(instances
-			(project "Modul_LCD"
+			(project "Modul_Main_Board"
 				(path "/e383a7f7-29ae-4aa9-abeb-7f7854670ab9"
 					(reference "H4")
@@
 		)
 		(instances
-			(project "Modul_LCD"
+			(project "Modul_Main_Board"
 				(path "/e383a7f7-29ae-4aa9-abeb-7f7854670ab9"
 					(reference "J7")
@@
 		)
 		(instances
-			(project "Modul_LCD"
+			(project "Modul_Main_Board"
 				(path "/e383a7f7-29ae-4aa9-abeb-7f7854670ab9"
 					(reference "J8")
@@
 		)
 		(instances
-			(project "Modul_LCD"
+			(project "Modul_Main_Board"
 				(path "/e383a7f7-29ae-4aa9-abeb-7f7854670ab9"
 					(reference "J5")
@@
 		)
 		(instances
-			(project "Modul_LCD"
+			(project "Modul_Main_Board"
 				(path "/e383a7f7-29ae-4aa9-abeb-7f7854670ab9"
 					(reference "J12")
@@
 			)
 		)
-		(property "Value" "1k"
+		(property "Value" "2k"
 			(at 26.67 31.75 90)
 			(effects
@@
 		)
 		(instances
-			(project "Modul_LCD"
+			(project "Modul_Main_Board"
 				(path "/e383a7f7-29ae-4aa9-abeb-7f7854670ab9"
 					(reference "R1")
@@
 		)
 		(instances
-			(project "Modul_LCD"
+			(project "Modul_Main_Board"
 				(path "/e383a7f7-29ae-4aa9-abeb-7f7854670ab9"
 					(reference "C1")
@@
 		)
 		(instances
-			(project "Modul_LCD"
+			(project "Modul_Main_Board"
 				(path "/e383a7f7-29ae-4aa9-abeb-7f7854670ab9"
 					(reference "J4")
